Commit message: Holiday release of Astrobee Robot Software.

File: simulation/astrobee_description/urdf/astrobee.urdf.xacro (robot description, xacro)
@@ -17,19 +17,31 @@
 <!-- permissions and limitations under the License.                          -->
 <robot name="astrobee" xmlns:xacro="http://www.ros.org/wiki/xacro">
+  <!-- Base platform -->
   <xacro:include filename="$(find astrobee_description)/urdf/astrobee_body.urdf.xacro" />
+  <!-- Modify the platform based on the world -->
+  <xacro:property name="ace" value="$(arg world)"/>
+  <xacro:if value="${ace == 'granite'}">
+    <xacro:include filename="$(find astrobee_description)/urdf/astrobee_carriage.urdf.xacro" />
+    <xacro:include filename="$(find astrobee_description)/urdf/macro_perching_arm.urdf.xacro" />
+    <xacro:perching_arm bay="top_aft" xyz="-0.01 0.0 -0.065" rpy="0.0 3.1415 0.0" />
+  </xacro:if>
+  <xacro:if value="${ace == 'iss'}">
+    <xacro:include filename="$(find astrobee_description)/urdf/macro_perching_arm.urdf.xacro" />
+    <xacro:perching_arm bay="top_aft" xyz="-0.01 0.0 -0.065" rpy="0.0 3.1415 0.0" />
+  </xacro:if>
+  <!-- Base model plugins -->
   <xacro:include filename="$(find astrobee_description)/urdf/model_pmc.urdf.xacro" />
-  <xacro:include filename="$(find astrobee_description)/urdf/model_drag.urdf.xacro" />
   <xacro:include filename="$(find astrobee_description)/urdf/model_truth.urdf.xacro" />
-  <!--
-  <xacro:include filename="$(find astrobee_description)/urdf/model_perching_arm.urdf.xacro" />
-  -->
   <xacro:include filename="$(find astrobee_description)/urdf/model_laser.urdf.xacro" />
   <xacro:include filename="$(find astrobee_description)/urdf/model_flashlights.urdf.xacro" />
+  <!-- Aerodynamics -->
+  <!--
+  <xacro:include filename="$(find astrobee_description)/urdf/model_drag.urdf.xacro" />
+  -->
+  <!-- Base Sensor plugins -->
   <xacro:include filename="$(find astrobee_description)/urdf/sensor_imu.urdf.xacro" />
   <xacro:include filename="$(find astrobee_description)/urdf/sensor_nav_cam.urdf.xacro" />
   <xacro:include filename="$(find astrobee_description)/urdf/sensor_dock_cam.urdf.xacro" />
-  <!--
   <xacro:include filename="$(find astrobee_description)/urdf/sensor_haz_cam.urdf.xacro" />
   <xacro:include filename="$(find astrobee_description)/urdf/sensor_perch_cam.urdf.xacro" />
-  -->
 </robot>

File: simulation/astrobee_description/urdf/sensor_dock_cam.urdf.xacro (robot description, xacro)
@@ -21,8 +21,8 @@
       <pose>0 0 0 0 0 0</pose>
       <always_on>0</always_on>
-      <update_rate>1</update_rate>
+      <update_rate>3</update_rate>
       <visualize>0</visualize>
       <camera>
-        <horizontal_fov>2.87507641955055</horizontal_fov> <!-- 130 degrees -->
+        <horizontal_fov>2.87507641955055</horizontal_fov>
         <image>
           <width>320</width>
@@ -31,5 +31,5 @@
         </image>
         <clip>
-          <near>0.2</near>
+          <near>0.03</near>
           <far>10</far>
         </clip>

File: simulation/astrobee_description/urdf/sensor_haz_cam.urdf.xacro (robot description, xacro)
@@ -21,5 +21,5 @@
       <pose>0 0 0 0 0 0</pose>
       <always_on>1</always_on>
-      <update_rate>1</update_rate>
+      <update_rate>5</update_rate>
       <visualize>0</visualize>
       <camera>

File: simulation/astrobee_description/urdf/sensor_nav_cam.urdf.xacro (robot description, xacro)
@@ -22,5 +22,5 @@
       <pose>0 0 0 0 0 0</pose>
       <always_on>0</always_on>
-      <update_rate>1</update_rate>
+      <update_rate>3</update_rate>
       <visualize>0</visualize>
       <camera>
@@ -32,5 +32,5 @@
         </image>
         <clip>
-          <near>0.2</near>
+          <near>0.03</near>
           <far>10</far>
         </clip>
@@ -45,5 +45,5 @@
       <pose>0 0 0 0 0 0</pose>
       <always_on>0</always_on>
-      <update_rate>2</update_rate>
+      <update_rate>5</update_rate>
       <visualize>0</visualize>
       <camera>
@@ -55,5 +55,5 @@
         </image>
         <clip>
-          <near>0.2</near>
+          <near>0.03</near>
           <far>10</far>
         </clip>

File: simulation/astrobee_description/urdf/sensor_perch_cam.urdf.xacro (robot description, xacro)
@@ -21,5 +21,5 @@
       <pose>0 0 0 0 0 0</pose>
       <always_on>1</always_on>
-      <update_rate>1</update_rate>
+      <update_rate>5</update_rate>
       <visualize>0</visualize>
       <camera>
