Commit message: Release v0.10.2.
* Perching behavior implemented
* Localization sparse mapping timeout increased to 10 minutes
* Already there tolerances decreased to allow for smaller moves
* Other minor bug fixes/software improvements

File: description/description/urdf/macro_perching_arm.urdf.xacro (robot description, xacro)
@@ -18,4 +18,7 @@
 <robot xmlns:xacro="http://www.ros.org/wiki/xacro">
   <xacro:macro name="perching_arm" params="bay xyz rpy">
+    <xacro:property name="prox_effort" value="1.0"/>
+    <xacro:property name="dist_effort" value="1.0"/>
+    <xacro:property name="grip_effort" value="0.1"/>
     <link name="${bay}">
       <self_collide>false</self_collide>
@@ -42,5 +45,4 @@
             filename="package://astrobee_freeflyer/meshes/base_link.dae" />
         </geometry>
-        <material name="${bay}_beige" />
       </visual>
       <collision>
@@ -88,5 +90,4 @@
             filename="package://astrobee_freeflyer/meshes/arm_proximal_link.dae" />
         </geometry>
-        <material name="${bay}_beige" />
       </visual>
       <collision>
@@ -112,5 +113,5 @@
         xyz="0 -1 0" />
       <limit
-        effort="2.7"
+        effort="${prox_effort}"
         lower="-2.0944"
         upper="1.57079"
@@ -141,5 +142,4 @@
             filename="package://astrobee_freeflyer/meshes/arm_distal_link.dae" />
         </geometry>
-        <material name="${bay}_beige" />
       </visual>
       <collision>
@@ -165,5 +165,5 @@
         xyz="0 0 1" />
       <limit
-        effort="2.7"
+        effort="${dist_effort}"
         lower="-1.57079"
         upper="1.57079"
@@ -194,5 +194,4 @@
             filename="package://astrobee_freeflyer/meshes/gripper_left_proximal_link.dae" />
         </geometry>
-        <material name="${bay}_beige" />
       </visual>
       <collision>
@@ -218,5 +217,5 @@
         xyz="0 0 1" />
       <limit
-        effort="0.1225"
+        effort="${grip_effort}"
         lower="0.349066"
         upper="0.698132"
@@ -247,5 +246,4 @@
             filename="package://astrobee_freeflyer/meshes/gripper_left_distal_link.dae" />
         </geometry>
-        <material name="${bay}_beige" />
       </visual>
       <collision>
@@ -271,5 +269,5 @@
         xyz="0 0 1" />
       <limit
-        effort="0.1225"
+        effort="${grip_effort}"
         lower="-1.22173"
         upper="-0.69813"
@@ -300,5 +298,4 @@
             filename="package://astrobee_freeflyer/meshes/gripper_right_proximal_link.dae" />
         </geometry>
-        <material name="${bay}_beige" />
       </visual>
       <collision>
@@ -324,5 +321,5 @@
         xyz="0 0 1" />
       <limit
-        effort="0.1225"
+        effort="${grip_effort}"
         lower="-0.698132"
         upper="-0.349066"
@@ -353,5 +350,4 @@
             filename="package://astrobee_freeflyer/meshes/gripper_right_distal_link.dae" />
         </geometry>
-        <material name="${bay}_beige" />
       </visual>
       <collision>
@@ -377,33 +373,9 @@
         xyz="0 0 1" />
       <limit
-        effort="0.1225"
+        effort="${grip_effort}"
         lower="0.69813"
         upper="1.22173"
         velocity="0.12" />
     </joint>
-    <material name="${bay}_beige">
-      <texture filename="package://astrobee_freeflyer/media/materials/textures/beige.png" />
-    </material>
-    <gazebo reference="${bay}">
-      <material>Astrobee/Beige</material>
-    </gazebo>
-    <gazebo reference="${bay}_arm_proximal_link">
-      <material>Astrobee/Beige</material>
-    </gazebo>
-    <gazebo reference="${bay}_arm_distal_link">
-      <material>Astrobee/Beige</material>
-    </gazebo>
-    <gazebo reference="${bay}_gripper_left_proximal_link">
-      <material>Astrobee/Beige</material>
-    </gazebo>
-    <gazebo reference="${bay}_gripper_left_distal_link">
-      <material>Astrobee/Beige</material>
-    </gazebo>
-    <gazebo reference="${bay}_gripper_right_proximal_link">
-      <material>Astrobee/Beige</material>
-    </gazebo>
-    <gazebo reference="${bay}_gripper_right_distal_link">
-      <material>Astrobee/Beige</material>
-    </gazebo>
     <gazebo>
       <plugin name="${bay}_perching_arm_ros" filename="libgazebo_model_plugin_perching_arm.so">
@@ -415,4 +387,5 @@
       </plugin>
     </gazebo>
+  -->
   </xacro:macro>
 </robot>

File: description/description/urdf/sensor_perch_cam.urdf.xacro (robot description, xacro)
@@ -37,6 +37,5 @@
         </depth_camera>
       </camera>
-      <plugin name="perch_cam_ros"
-              filename="libgazebo_sensor_plugin_perch_cam.so"/>
+      <plugin name="perch_cam_ros" filename="libgazebo_sensor_plugin_perch_cam.so"/>
     </sensor>
   </gazebo>

Commit message: fixing noetic prefix

File: description/description/urdf/macro_perching_arm.urdf.xacro (robot description, xacro)
@@ -21,5 +21,5 @@
     <xacro:property name="dist_effort" value="1.0"/>
     <xacro:property name="grip_effort" value="0.1"/>
-    <link name="${bay}">
+    <link name="${prefix}${bay}">
       <self_collide>false</self_collide>
       <inertial>
@@ -62,9 +62,9 @@
         rpy="${rpy}" />
       <parent
-        link="body" />
-      <child
-        link="${bay}" />
-    </joint>
-    <link name="${bay}_arm_proximal_link">
+        link="${prefix}body" />
+      <child
+        link="${prefix}${bay}" />
+    </joint>
+    <link name="${prefix}${bay}_arm_proximal_link">
       <self_collide>false</self_collide>
       <inertial>
@@ -107,7 +107,7 @@
         rpy="0 1.57079632679 0" />
       <parent
-        link="${bay}" />
-      <child
-        link="${bay}_arm_proximal_link" />
+        link="${prefix}${bay}" />
+      <child
+        link="${prefix}${bay}_arm_proximal_link" />
       <axis
         xyz="0 -1 0" />
@@ -118,5 +118,5 @@
         velocity="0.12" />
     </joint>
-    <link name="${bay}_arm_distal_link">
+    <link name="${prefix}${bay}_arm_distal_link">
       <self_collide>false</self_collide>
       <inertial>
@@ -159,7 +159,7 @@
         rpy="0 0 0" />
       <parent
-        link="${bay}_arm_proximal_link" />
-      <child
-        link="${bay}_arm_distal_link" />
+        link="${prefix}${bay}_arm_proximal_link" />
+      <child
+        link="${prefix}${bay}_arm_distal_link" />
       <axis
         xyz="0 0 1" />
@@ -170,5 +170,5 @@
         velocity="0.12" />
     </joint>
-    <link name="${bay}_gripper_left_proximal_link">
+    <link name="${prefix}${bay}_gripper_left_proximal_link">
       <self_collide>false</self_collide>
       <inertial>
@@ -211,7 +211,7 @@
         rpy="0 0 0" />
       <parent
-        link="${bay}_arm_distal_link" />
-      <child
-        link="${bay}_gripper_left_proximal_link" />
+        link="${prefix}${bay}_arm_distal_link" />
+      <child
+        link="${prefix}${bay}_gripper_left_proximal_link" />
       <axis
         xyz="0 0 1" />
@@ -222,5 +222,5 @@
         velocity="0.12" />
     </joint>
-    <link name="${bay}_gripper_left_distal_link">
+    <link name="${prefix}${bay}_gripper_left_distal_link">
       <self_collide>false</self_collide>
       <inertial>
@@ -263,7 +263,7 @@
         rpy="0 0 0" />
       <parent
-        link="${bay}_gripper_left_proximal_link" />
-      <child
-        link="${bay}_gripper_left_distal_link" />
+        link="${prefix}${bay}_gripper_left_proximal_link" />
+      <child
+        link="${prefix}${bay}_gripper_left_distal_link" />
       <axis
         xyz="0 0 1" />
@@ -274,5 +274,5 @@
         velocity="0.12" />
     </joint>
-    <link name="${bay}_gripper_right_proximal_link">
+    <link name="${prefix}${bay}_gripper_right_proximal_link">
       <self_collide>false</self_collide>
       <inertial>
@@ -315,7 +315,7 @@
         rpy="0 0 0" />
       <parent
-        link="${bay}_arm_distal_link" />
-      <child
-        link="${bay}_gripper_right_proximal_link" />
+        link="${prefix}${bay}_arm_distal_link" />
+      <child
+        link="${prefix}${bay}_gripper_right_proximal_link" />
       <axis
         xyz="0 0 1" />
@@ -326,5 +326,5 @@
         velocity="0.12" />
     </joint>
-    <link name="${bay}_gripper_right_distal_link">
+    <link name="${prefix}${bay}_gripper_right_distal_link">
       <self_collide>false</self_collide>
       <inertial>
@@ -367,7 +367,7 @@
         rpy="0 0 0" />
       <parent
-        link="${bay}_gripper_right_proximal_link" />
-      <child
-        link="${bay}_gripper_right_distal_link" />
+        link="${prefix}${bay}_gripper_right_proximal_link" />
+      <child
+        link="${prefix}${bay}_gripper_right_distal_link" />
       <axis
         xyz="0 0 1" />
@@ -388,5 +388,4 @@
       </plugin>
     </gazebo>
-  -->
   </xacro:macro>
 </robot>

File: description/description/urdf/model.urdf.xacro (robot description, xacro)
@@ -23,6 +23,7 @@
   <xacro:property name="pay_bot_front" value="$(arg bot_front)"/>
   <xacro:property name="ns" value="$(arg ns)"/>
+  <xacro:property name="prefix" value="$(arg prefix)"/>
   <!-- BASE GEOMETRY -->
- <link name="body">
+ <link name="${prefix}body">
     <self_collide>false</self_collide>
     <!-- body -->
@@ -91,5 +92,5 @@
   </link>
   <!-- This is a workaround for KDL -->
-  <link name="inertial_link">
+  <link name="${prefix}inertial_link">
     <self_collide>false</self_collide>
     <inertial>
@@ -101,6 +102,6 @@
   <joint name="inertial_joint" type="fixed">
     <origin xyz="0 0 0" rpy="0 0 0" />
-    <parent link="body" />
-    <child link="inertial_link" />
+    <parent link="${prefix}body" />
+    <child link="${prefix}inertial_link" />
   </joint>
   <!-- MODEL -->

File: description/description/urdf/sensor_dock_cam.urdf.xacro (robot description, xacro)
@@ -17,5 +17,5 @@
 <!-- permissions and limitations under the License.                          -->
 <robot xmlns:xacro="http://www.ros.org/wiki/xacro">
-  <gazebo reference="body">
+  <gazebo reference="${prefix}body">
     <sensor name="dock_cam" type="wideanglecamera">
       <pose>0 0 0 0 0 0</pose>

File: description/description/urdf/sensor_haz_cam.urdf.xacro (robot description, xacro)
@@ -17,5 +17,5 @@
 <!-- permissions and limitations under the License.                          -->
 <robot xmlns:xacro="http://www.ros.org/wiki/xacro">
-  <gazebo reference="body">
+  <gazebo reference="${prefix}body">
     <sensor name="haz_cam" type="depth">
       <pose>0 0 0 0 0 0</pose>

File: description/description/urdf/sensor_imu.urdf.xacro (robot description, xacro)
@@ -17,5 +17,5 @@
 <!-- permissions and limitations under the License.                          -->
 <robot xmlns:xacro="http://www.ros.org/wiki/xacro">
-  <gazebo reference="body">
+  <gazebo reference="${prefix}body">
     <sensor name="imu" type="imu">
       <pose>0 0 0 0 0 0</pose>

File: description/description/urdf/sensor_nav_cam.urdf.xacro (robot description, xacro)
@@ -17,5 +17,5 @@
 <!-- permissions and limitations under the License.                          -->
 <robot xmlns:xacro="http://www.ros.org/wiki/xacro">
-  <gazebo reference="body">
+  <gazebo reference="${prefix}body">
     <sensor name="nav_cam" type="wideanglecamera">
       <pose>0 0 0 0 0 0</pose>

File: description/description/urdf/sensor_perch_cam.urdf.xacro (robot description, xacro)
@@ -17,5 +17,5 @@
 <!-- permissions and limitations under the License.                          -->
 <robot xmlns:xacro="http://www.ros.org/wiki/xacro">
-  <gazebo reference="body">
+  <gazebo reference="${prefix}body">
     <sensor name="perch_cam" type="depth">
       <pose>0 0 0 0 0 0</pose>

File: description/description/urdf/sensor_sci_cam.urdf.xacro (robot description, xacro)
@@ -17,5 +17,5 @@
 <!-- permissions and limitations under the License.                          -->
 <robot xmlns:xacro="http://www.ros.org/wiki/xacro">
-  <gazebo reference="body">
+  <gazebo reference="${prefix}body">
     <sensor name="sci_cam" type="camera">
       <pose>0 0 0 0 0 0</pose>
