Commit message: Release 0.7.6. Code on flight units.

File: description/description/urdf/model.urdf.xacro (robot description, xacro)
@@ -94,7 +94,7 @@
     <self_collide>false</self_collide>
     <inertial>
-      <mass value="7.0"/>
+      <mass value="9.176"/>
       <origin xyz="0 0 0"/>
-      <inertia ixx="0.1083" ixy="0.0" ixz="0.0" iyy="0.1083" iyz="0.0" izz="0.1083"/>
+      <inertia ixx="0.1873" ixy="0.0" ixz="0.0" iyy="0.1873" iyz="0.0" izz="0.1873"/>
     </inertial>
   </link>
@@ -111,4 +111,8 @@
   <xacro:include filename="$(find description)/urdf/model_laser.urdf.xacro" />
   <xacro:include filename="$(find description)/urdf/model_flashlights.urdf.xacro" />
+  <xacro:include filename="$(find description)/urdf/model_speed_cam.urdf.xacro" />
+  <xacro:include filename="$(find description)/urdf/model_signal_lights.urdf.xacro" />
+  <!-- Monitors -->
+  <xacro:include filename="$(find description)/urdf/model_monitors.urdf.xacro" />
   <!-- SENSORS -->
   <xacro:include filename="$(find description)/urdf/sensor_imu.urdf.xacro" />

File: description/description/urdf/model_carriage.urdf.xacro (robot description, xacro)
@@ -19,7 +19,7 @@
   <link name="carriage">
     <inertial>
-      <mass value="4.0"/>
+      <mass value="9.724"/>
       <origin xyz="0 0 -0.02"/>
-      <inertia ixx="0.1083" ixy="0.0" ixz="0.0" iyy="0.1083" iyz="0.0" izz="0.1083"/>
+      <inertia ixx="0.694860833" ixy="0.0" ixz="0.0" iyy="0.694860833" iyz="0.0" izz="0.595595"/>
     </inertial>
     <visual name="carriage_visual">

File: description/description/urdf/model_pmc.urdf.xacro (robot description, xacro)
@@ -20,4 +20,5 @@
     <plugin name="pmc_ros" filename="libgazebo_model_plugin_pmc.so">
       <rate>62.5</rate>
+      <bypass_blower_model>true</bypass_blower_model>
     </plugin>
   </gazebo>

Commit message: Release v0.8.0.
Many improvements and fixes (see RELEASE.md).

File: description/description/urdf/model.urdf.xacro (robot description, xacro)
@@ -94,7 +94,7 @@
     <self_collide>false</self_collide>
     <inertial>
-      <mass value="9.176"/>
+      <mass value="9.0877"/>
       <origin xyz="0 0 0"/>
-      <inertia ixx="0.1873" ixy="0.0" ixz="0.0" iyy="0.1873" iyz="0.0" izz="0.1873"/>
+      <inertia ixx="0.1454" ixy="0.0" ixz="0.0" iyy="0.1366" iyz="0.0" izz="0.1594"/>
     </inertial>
   </link>

File: description/description/urdf/model_carriage.urdf.xacro (robot description, xacro)
@@ -19,7 +19,8 @@
   <link name="carriage">
     <inertial>
-      <mass value="9.724"/>
+      <mass value="9.8838"/>
       <origin xyz="0 0 -0.02"/>
-      <inertia ixx="0.694860833" ixy="0.0" ixz="0.0" iyy="0.694860833" iyz="0.0" izz="0.595595"/>
+      <!-- ixx and iyy are dummy values                        -->
+      <inertia ixx="0.694860833" ixy="0.0" ixz="0.0" iyy="0.694860833" iyz="0.0" izz="0.0923"/>
     </inertial>
     <visual name="carriage_visual">

File: description/description/urdf/model_pmc.urdf.xacro (robot description, xacro)
@@ -20,5 +20,5 @@
     <plugin name="pmc_ros" filename="libgazebo_model_plugin_pmc.so">
       <rate>62.5</rate>
-      <bypass_blower_model>true</bypass_blower_model>
+      <bypass_blower_model>false</bypass_blower_model>
     </plugin>
   </gazebo>

Commit message: not adding / in case of no prefix

File: description/description/urdf/model.urdf.xacro (robot description, xacro)
@@ -24,4 +24,7 @@
   <xacro:property name="ns" value="$(arg ns)"/>
   <xacro:property name="prefix" value="$(arg prefix)"/>
+  <xacro:if value="${prefix == '/'}">
+    <xacro:property name="prefix" value=""/>
+  </xacro:if>
   <!-- BASE GEOMETRY -->
  <link name="${prefix}body">

Commit message: Fix tf prefix noetic (#213)
* fixing noetic prefix
* not adding / in case of no prefix
* taking out the prefix from robots for rviz visuaization

File: description/description/urdf/model.urdf.xacro (robot description, xacro)
@@ -23,6 +23,10 @@
   <xacro:property name="pay_bot_front" value="$(arg bot_front)"/>
   <xacro:property name="ns" value="$(arg ns)"/>
+  <xacro:property name="prefix" value="$(arg prefix)"/>
+  <xacro:if value="${prefix == '/'}">
+    <xacro:property name="prefix" value=""/>
+  </xacro:if>
   <!-- BASE GEOMETRY -->
- <link name="body">
+ <link name="${prefix}body">
     <self_collide>false</self_collide>
     <!-- body -->
@@ -91,5 +95,5 @@
   </link>
   <!-- This is a workaround for KDL -->
-  <link name="inertial_link">
+  <link name="${prefix}inertial_link">
     <self_collide>false</self_collide>
     <inertial>
@@ -101,6 +105,6 @@
   <joint name="inertial_joint" type="fixed">
     <origin xyz="0 0 0" rpy="0 0 0" />
-    <parent link="body" />
-    <child link="inertial_link" />
+    <parent link="${prefix}body" />
+    <child link="${prefix}inertial_link" />
   </joint>
   <!-- MODEL -->
