Commit message: fixing carriage tf prefix

File: description/description/urdf/model_carriage.urdf.xacro (robot description, xacro)
@@ -17,5 +17,5 @@
 <!-- permissions and limitations under the License.                          -->
 <robot xmlns:xacro="http://www.ros.org/wiki/xacro">
-  <link name="carriage">
+  <link name="${prefix}carriage">
     <inertial>
       <mass value="9.8838"/>
@@ -44,7 +44,7 @@
       rpy="0 0 0" />
     <parent
-      link="body" />
+      link="${prefix}body" />
     <child
-      link="carriage" />
+      link="${prefix}carriage" />
   </joint>
   <gazebo reference="carriage">
