Commit message: feat: adding discower world with new platform

File: description/discower/urdf/model.urdf.xacro (robot description, xacro)
@@ -34,61 +34,11 @@
       <origin xyz="0 0 0" rpy="0 0 0" />
       <geometry>
-        <mesh filename="package://astrobee_freeflyer/meshes/body.dae"/>
+        <mesh filename="package://discower_platforms/meshes/proto.dae"/>
       </geometry>
     </visual>
     <collision name="body_collision">
-      <origin xyz="-0.000794 0.000229 -0.003907" rpy="0 0 0" />
+      <origin xyz="0 0 0.25" rpy="0 0 0" />
       <geometry>
-        <box size="0.290513 0.151942 0.281129" />
-      </geometry>
-    </collision>
-    <!-- port pmc -->
-    <visual name="pmc_port_visual">
-      <origin xyz="0 0 0" rpy="0 0 0" />
-      <geometry>
-        <mesh filename="package://astrobee_freeflyer/meshes/pmc.dae"/>
-      </geometry>
-    </visual>
-    <visual name="pmc_port_bumper_visual">
-      <origin xyz="0 0 0" rpy="0 0 0" />
-      <geometry>
-        <mesh filename="package://astrobee_freeflyer/meshes/pmc_bumper.dae"/>
-      </geometry>
-    </visual>
-    <visual name="pmc_port_skin_visual">
-      <origin xyz="0 0 0" rpy="0 0 0" />
-      <geometry>
-        <mesh filename="package://astrobee_freeflyer/meshes/pmc_skin${ns}.dae"/>
-      </geometry>
-    </visual>
-    <collision name="pmc_port_collision">
-      <origin xyz="0 -0.117546 0" rpy="0 0 0" />
-      <geometry>
-        <box size="0.319199 0.083962 0.319588" />
-      </geometry>
-    </collision>
-    <!-- starboard pmc -->
-    <visual name="pmc_stbd_visual">
-      <origin xyz="0 0 0" rpy="0 3.14 3.14" />
-      <geometry>
-        <mesh filename="package://astrobee_freeflyer/meshes/pmc.dae"/>
-      </geometry>
-    </visual>
-    <visual name="pmc_stbd_bumper_visual">
-      <origin xyz="0 0 0" rpy="0 3.14 3.14" />
-      <geometry>
-        <mesh filename="package://astrobee_freeflyer/meshes/pmc_bumper.dae"/>
-      </geometry>
-    </visual>
-    <visual name="pmc_stbd_skin_visual">
-      <origin xyz="0 0 0" rpy="0 3.14 3.14" />
-      <geometry>
-        <mesh filename="package://astrobee_freeflyer/meshes/pmc_skin${ns}.dae"/>
-      </geometry>
-    </visual>
-    <collision name="pmc_stbd_collision">
-      <origin xyz="0 0.117546 0" rpy="0 0 0" />
-      <geometry>
-        <box size="0.319199 0.083962 0.319588" />
+        <cylinder length="0.5" radius="0.2"/>
       </geometry>
     </collision>
@@ -98,6 +48,6 @@
     <self_collide>false</self_collide>
     <inertial>
-      <mass value="9.0877"/>
-      <origin xyz="0 0 0"/>
+      <mass value="12.5"/>
+      <origin xyz="0 0 0.2"/>
       <inertia ixx="0.1454" ixy="0.0" ixz="0.0" iyy="0.1366" iyz="0.0" izz="0.1594"/>
     </inertial>
@@ -108,40 +58,11 @@
     <child link="${prefix}inertial_link" />
   </joint>
-  <!-- MODEL -->
+  <!-- MODEL-->
   <xacro:include filename="$(find discower_description)/urdf/model_drag.urdf.xacro" />
   <xacro:include filename="$(find discower_description)/urdf/model_pmc.urdf.xacro" />
-  <xacro:include filename="$(find discower_description)/urdf/model_eps.urdf.xacro" />
   <xacro:include filename="$(find discower_description)/urdf/model_truth.urdf.xacro" />
-  <xacro:include filename="$(find discower_description)/urdf/model_laser.urdf.xacro" />
-  <xacro:include filename="$(find discower_description)/urdf/model_flashlights.urdf.xacro" />
   <xacro:include filename="$(find discower_description)/urdf/model_speed_cam.urdf.xacro" />
-  <xacro:include filename="$(find discower_description)/urdf/model_signal_lights.urdf.xacro" />
   <!-- <xacro:include filename="$(find discower_description)/urdf/model_sitl.urdf.xacro" /> -->
-  <!-- Monitors -->
-  <xacro:include filename="$(find discower_description)/urdf/model_monitors.urdf.xacro" />
   <!-- SENSORS -->
   <xacro:include filename="$(find discower_description)/urdf/sensor_imu.urdf.xacro" />
-  <xacro:include filename="$(find discower_description)/urdf/sensor_nav_cam.urdf.xacro" />
-  <xacro:include filename="$(find discower_description)/urdf/sensor_dock_cam.urdf.xacro" />
-  <xacro:include filename="$(find discower_description)/urdf/sensor_haz_cam.urdf.xacro" />
-  <xacro:include filename="$(find discower_description)/urdf/sensor_perch_cam.urdf.xacro" />
-  <!-- PERCHING ARM -->
-  <xacro:include filename="$(find discower_description)/urdf/macro_perching_arm.urdf.xacro" />
-  <xacro:if value="${pay_top_aft == 'perching_arm'}">
-    <xacro:perching_arm bay="top_aft"
-                        xyz="-0.01 0.0 -0.065"
-                        rpy="0.0 3.1415 0.0" />
-  </xacro:if>
-  <xacro:if value="${pay_bot_aft == 'perching_arm'}">
-    <xacro:perching_arm bay="bot_aft"
-                        xyz="-0.01 0.0 -0.065"
-                        rpy="0.0 3.1415 0.0" />
-  </xacro:if>
-  <xacro:if value="${pay_bot_front == 'perching_arm'}">
-    <xacro:perching_arm bay="bot_aft"
-                        xyz="-0.01 0.0 -0.065"
-                        rpy="0.0 3.1415 0.0" />
-  </xacro:if>
-  <!-- GRANITE-SPECIFIC OPTIONS -->
-  <xacro:include filename="$(find discower_description)/urdf/model_carriage.urdf.xacro" />
 </robot>
